Commit message: partially cleaned up launch files

File: omni_bot/description/depth_camera.xacro (robot description, xacro)
@@ -16,10 +16,10 @@
     <joint name="camera_optical_joint" type="fixed">
         <parent link="camera_link"/>
-        <child link="camera_link_optical"/>
+        <child link="camera_color_optical_frame"/>
         <origin xyz="0 0 0" rpy="${-pi/2} 0 ${-pi/2}"/>
     </joint>
-    <link name="camera_link_optical">
+    <link name="camera_color_optical_frame">
     </link>
-    <gazebo reference="camera_link_optical">
+    <gazebo reference="camera_color_optical_frame">
         <material>Gazebo/Red</material>
         <!--
@@ -73,5 +73,5 @@
             <visualize>1</visualize>
             <pose>0 0 0 0 -0 0</pose>
-            <topic>camera/image_raw</topic>
+            <topic>camera/camera/color/image_raw</topic>
             <gz_frame_id>camera_link_optical</gz_frame_id>
             <camera name="d435">
@@ -97,5 +97,5 @@
             <update_rate>15</update_rate>
             <visualize>0</visualize>
-            <topic>camera/depth/image_raw</topic>
+            <topic>camera/camera/aligned_depth_to_color/image_raw</topic>
             <pose>0 0 0 0 -0 0</pose>
             <gz_frame_id>camera_link_optical</gz_frame_id>
